File: hillside46/hillside46.kicad_sch (KiCad schematic)
At the start: 92 parts, among them J1 Haptic, J2 TRRS, J3 Bat_Pos, J4 Bat_Neg, J5 Bat_Pos, J6 Bat_Neg, K1 SW_Key, K10 SW_Key, K11 SW_Key, K12 SW_Key, K13 SW_Key, K14 SW_Key, K15 SW_Key, K16 SW_Key, K17 SW_Key, K18 SW_Key, K19 SW_Rotary, K2 SW_Key, K20 SW_Rotary, K21 SW_Key, K22 SW_Key, K23 SW_Key, K3 SW_Key, K4 SW_Key, K5 SW_Key, K6 SW_Key, K7 SW_Key, K8 SW_Key, K9 SW_Key, SW1 SKQGAFE010, SW2 SW_Power, U1 ProMicro_r, U2 SRV05-4

Commit message: my mods
Parts:
- removed D1, D2, D3, D4: SK6812-MINI-E, hillside_basic:SK6812-MINI-E, symbol hillside_basic:SK6812-MINI-E
- removed D10, D11, D12, D13, D14, D15, D19, D20, D21, D7, D8, D9: BAV70, hillside_basic:SOT-23, symbol hillside_basic:BAV70_Small
- removed H1: Mount_Tenting, hillside:Tenting_Puck, symbol hillside:Mount_Tenting
- removed H26, H27, H28, H29, H30, H31: Breakoff Hole, hillside_basic:HoleBreakoff_1mm, symbol Mechanical:MountingHole
- added D10, D11, D12, D13, D14, D15, D16, D17, D18, D22, D23, D24, D25, D26, D27, D28, D29, D30, D5, D6, D7, D8, D9: 1N4148W, Diode_SMD:D_SOD-123, symbol Diode:1N4148W
- K1, K10, K11, K12, K13, K14, K15, K16, K17, K18, K2, K21, K22, K23, K3, K4, K5, K6, K7, K8, K9: footprint hillside:pg1350-R_hotswap -> (none)
- K19, K20: value SW_Rotary -> SW_Key; footprint hillside:pg1350-DR_rotary_hotswap -> (none); symbol hillside:SW_Rotary -> hillside:SW_Key
Connections:
- net GND: no longer K19.C, K20.C
- net col1: now also K20.1; no longer K20.S1
- net col5: now also K19.1; no longer K19.S1
- net enc_a: no longer K19.A, K20.A
- net enc_b: no longer K19.B, K20.B
- net row0: now also D11.1 (K), D13.1 (K), D15.1 (K), D5.1 (K), D7.1 (K), D9.1 (K)
- net row1: now also D10.1 (K), D12.1 (K), D14.1 (K), D24.1 (K), D6.1 (K), D8.1 (K)
- net row2: now also D16.1 (K), D17.1 (K), D18.1 (K), D22.1 (K), D23.1 (K), D25.1 (K)
- net row3: now also JP2.2 (B), D26.1 (K), D27.1 (K), D28.1 (K), D29.1 (K), D30.1 (K)
- net at K13.2: now also D16.2 (A)
- net at K14.2: now also D17.2 (A)
- net at K23.2: now also D28.2 (A)
- net at K9.2: now also D10.2 (A)
- net at K10.2: now also D12.2 (A)
- net at K15.2: now also D18.2 (A)
- net at K16.2: now also D22.2 (A)
- net at K1.2: now also D5.2 (A)
- net at K2.2: now also D7.2 (A)
- net at K5.2: now also D13.2 (A)
- net at K6.2: now also D15.2 (A)
- net at K11.2: now also D14.2 (A)
- net at K12.2: now also D24.2 (A)
- net at K17.2: now also D23.2 (A)
- net at K18.2: now also D25.2 (A)
- net at K3.2: now also D9.2 (A)
- net at K4.2: now also D11.2 (A)
- net at K7.2: now also D6.2 (A)
- net at K8.2: now also D8.2 (A)
- net at K21.2: now also D26.2 (A)
- net at K22.2: now also D27.2 (A)
- new net: D30.2 (A), K20.2
- new net: D29.2 (A), K19.2
- no-connect marks 5 -> 4
Other:
- note removed: "Breakoff Holes"
- moved on the sheet: JP2, K1, K10, K11, K12, K13, K14, K15, K16, K17, K18, K2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

Commit message: trrs changes
Parts:
- removed H25: ToolingHole, hillside_basic:ToolingHole_1.152mm, symbol Mechanical:MountingHole
- removed H3: Logo, hillside:Hillside_Logo, symbol hillside:Logo
- removed J2: TRRS, hillside:MJ-4PP-9, symbol hillside:TRRS
- added J2: USB_C_Receptacle_USB2.0_16P, Package_DFN_QFN:WDFN-10-1EP_3x3mm_P0.5mm_EP1.8x2.5mm, symbol Connector:USB_C_Receptacle_USB2.0_16P
- added JP3, JP4: SolderJumper_3_Open, symbol Jumper:SolderJumper_3_Open
- D10, D11, D12, D13, D14, D15, D16, D17, D18, D22, D23, D24, D25, D26, D27, D28, D29, D30, D5, D6, D7, D8, D9: footprint Diode_SMD:D_SOD-123 -> hillside:D_SOD-123_Hillside_reversable
Connections:
- net GND: now also J2.A1 (GND), J2.A12 (GND), J2.B1 (GND), J2.B12 (GND), J2.SH (SHIELD)
- net VCC: now also J2.A4 (VBUS), J2.A9 (VBUS), J2.B4 (VBUS), J2.B9 (VBUS)
- net LED renamed TX
- net TX: now also JP3.2 (C), JP4.2 (C)
- net data renamed RX
- net RX: now also JP3.3 (B), JP4.3 (B); no longer U2.6 (IO4)
- new net UART_A: J2.A7 (D-), J2.B7 (D-), JP4.1 (A), U2.6 (IO4)
- new net UART_B: J2.A6 (D+), J2.B6 (D+), JP3.1 (A), U2.1 (IO4)
- no-connect marks 4 -> 9
Other:
- moved on the sheet: C2, C3, SW1, U1

Commit message: usb-c switch changes
Parts:
- removed H10, H11, H12, H13, H14, H15, H16, H17, H18, H19, H2, H20, H21, H22, H8, H9: Bumpon, hillside:Bumpon, symbol hillside_basic:Bumpon
- removed H23, H24: ToolingHole, hillside_basic:ToolingHole_1.152mm, symbol Mechanical:MountingHole
- removed J2: USB_C_Receptacle_USB2.0_16P, Package_DFN_QFN:WDFN-10-1EP_3x3mm_P0.5mm_EP1.8x2.5mm, symbol Connector:USB_C_Receptacle_USB2.0_16P
- removed JP3, JP4: SolderJumper_3_Open, symbol Jumper:SolderJumper_3_Open
- removed V2: Via, hillside_basic:VIA-0.8mm, symbol hillside_basic:Via
- added J2: USB_C_Receptacle_PowerOnly_6P, hillside:USB_C_Receptacle_GCT_USB4125-xx-x-0190_6P_TopMnt_Horizontal, symbol Connector:USB_C_Receptacle_PowerOnly_6P
- K1, K2, K3, K4: footprint (none) -> hillside:pg1350-R_hotswap
- SW1: footprint hillside_basic:SW_SPST_SKQG_WithStem -> hillside:SW_Push_1P1T_NO_CK_KMR2
- SW2: footprint hillside_basic:SW_SPDT_JS202011AQN -> hillside:SW_SPDT_Shouhan_MSK12C02
Connections:
- net UART_A is gone; now on net data: U2.6 (IO4)
- net GND: now also J2.A12 (GND), J2.B12 (GND), J2.SH (SHIELD)
- net VCC: now also J2.A9 (VBUS), J2.B9 (VBUS)
- net RX renamed data
- net data: now also J2.A5 (CC1), J2.B5 (CC2)
- net TX renamed led
- net UART_B: no longer names the net of U2.1 (IO4)
- no-connect marks 9 -> 6
Other:
- note removed: "Mounts under Board"
- note removed: "PCB Assembly"
